Commit message: fix: urdf issues

File: spot/util/pybullet_data/assets/urdf/spot.urdf (robot description, URDF)
Before this commit: robot spot, 24 links, 23 joints
Links:
- link back: geometry collision box size=0.114 0.075 0.085; visual mesh filename=package://spot/util/pybullet_data/assets/urdf/stl/OpenQuadr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 scale=1 1 1
- link back_bracket: geometry collision box size=0.025 0.075 0.085; visual mesh filename=package://spot/util/pybullet_data/assets/urdf/stl/OpenQuadr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 scale=1 1 1
- link back_left_foot: geometry collision mesh filename=package://spot/util/pybullet_data/assets/urdf/stl/OpenQuadr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 scale=1 1 1; visual mesh filename=package://spot/util/pybullet_data/assets/urdf/stl/OpenQuadr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 scale=1 1 1
- link back_left_hip: geometry collision box size=0.05 0.065 0.065; visual mesh filename=package://spot/util/pybullet_data/assets/urdf/stl/OpenQuadr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 scale=1 1 1
- link back_left_lower_leg: geometry collision box size=0.035 0.035 0.12; visual mesh filename=package://spot/util/pybullet_data/assets/urdf/stl/OpenQuadr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 scale=1 1 1
- link back_left_upper_leg: geometry collision box size=0.035 0.035 0.11; visual mesh filename=package://spot/util/pybullet_data/assets/urdf/stl/OpenQuadr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 scale=1 1 1
- link back_right_foot: geometry collision mesh filename=package://spot/util/pybullet_data/assets/urdf/stl/OpenQuadr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 scale=1 1 1; visual mesh filename=package://spot/util/pybullet_data/assets/urdf/stl/OpenQuadr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 scale=1 1 1
- link back_right_hip: geometry collision box size=0.05 0.065 0.065; visual mesh filename=package://spot/util/pybullet_data/assets/urdf/stl/OpenQuadr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 scale=1 1 1
- link back_right_lower_leg: geometry collision box size=0.035 0.035 0.12; visual mesh filename=package://spot/util/pybullet_data/assets/urdf/stl/OpenQuadr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 scale=1 1 1
- link back_right_upper_leg: geometry collision box size=0.035 0.035 0.11; visual mesh filename=package://spot/util/pybullet_data/assets/urdf/stl/OpenQuadr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 scale=1 1 1
- link base_link: geometry collision box size=0.114 0.2 0.1; visual mesh filename=package://spot/util/pybullet_data/assets/urdf/stl/OpenQuadr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 scale=1 1 1
- link battery: geometry collision box size=0.048 0.145 0.026; visual mesh filename=package://spot/util/pybullet_data/assets/urdf/stl/OpenQuadr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 scale=1 1 1
- link chassis_left: geometry collision box size=0.06 0.15 0.006; visual mesh filename=package://spot/util/pybullet_data/assets/urdf/stl/OpenQuadr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 scale=1 1 1
- link chassis_right: geometry collision box size=0.06 0.15 0.006; visual mesh filename=package://spot/util/pybullet_data/assets/urdf/stl/OpenQuadr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 scale=1 1 1
- link front: geometry collision box size=0.114 0.045 0.085; visual mesh filename=package://spot/util/pybullet_data/assets/urdf/stl/OpenQuadr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 scale=1 1 1
- link front_bracket: geometry collision box size=0.025 0.075 0.085; visual mesh filename=package://spot/util/pybullet_data/assets/urdf/stl/OpenQuadr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 scale=1 1 1
- link front_left_foot: geometry collision mesh filename=package://spot/util/pybullet_data/assets/urdf/stl/OpenQuadr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 scale=1 1 1; visual mesh filename=package://spot/util/pybullet_data/assets/urdf/stl/OpenQuadr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 scale=1 1 1
- link front_left_hip: geometry collision box size=0.05 0.065 0.065; visual mesh filename=package://spot/util/pybullet_data/assets/urdf/stl/OpenQuadr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 scale=1 1 1
- link front_left_lower_leg: geometry collision box size=0.035 0.035 0.12; visual mesh filename=package://spot/util/pybullet_data/assets/urdf/stl/OpenQuadr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 scale=1 1 1
- link front_left_upper_leg: geometry collision box size=0.035 0.035 0.11; visual mesh filename=package://spot/util/pybullet_data/assets/urdf/stl/OpenQuadr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 scale=1 1 1
- link front_right_foot: geometry collision mesh filename=package://spot/util/pybullet_data/assets/urdf/stl/OpenQuadr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 scale=1 1 1; visual mesh filename=package://spot/util/pybullet_data/assets/urdf/stl/OpenQuadr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 scale=1 1 1
- link front_right_hip: geometry collision box size=0.05 0.065 0.065; visual mesh filename=package://spot/util/pybullet_data/assets/urdf/stl/OpenQuadr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 scale=1 1 1
- link front_right_lower_leg: geometry collision box size=0.035 0.035 0.12; visual mesh filename=package://spot/util/pybullet_data/assets/urdf/stl/OpenQuadr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 scale=1 1 1
- link front_right_upper_leg: geometry collision box size=0.035 0.035 0.11; visual mesh filename=package://spot/util/pybullet_data/assets/urdf/stl/OpenQuadr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 scale=1 1 1
